Commit message: scaled the bot down

File: src/bme_gazebo_sensors/urdf/mogi_bot.urdf (robot description, URDF)
Before this commit: robot mogi_bot, 8 links, 7 joints
Links:
- link base_link: geometry collision box size=1.6 .8 .4; collision sphere radius=0.19975
- link camera_link: geometry collision box size=.12 .12 .12; visual box size=.12 .12 .12
- link left_wheel: geometry collision cylinder length=.2 radius=.4; visual mesh filename=package://bme_gazebo_sensors/meshes/wheel.dae scale=4 4 4
- link right_wheel: geometry collision cylinder length=.2 radius=.4; visual mesh filename=package://bme_gazebo_sensors/meshes/wheel.dae scale=4 4 4
- link scan_link: geometry collision box size=.4 .4 .4; visual mesh filename=package://bme_gazebo_sensors/meshes/lidar.dae scale=4 4 4
Joints:
- joint camera_joint: origin xyz=1.8 0 0.6 rpy=0 0 0 -> xyz=0.9 0 0.3 rpy=0 0 0
- joint camera_optical_joint: origin xyz=0 0 0 rpy=-1.5707 0 -1.5707 -> xyz=0 0 0 rpy=-0.78535 0 -0.78535
- joint left_wheel_joint: origin xyz=0 1.2 0 rpy=0 0 0 -> xyz=0 0.6 0 rpy=0 0 0
- joint right_wheel_joint: origin xyz=0 -1.2 0 rpy=0 0 0 -> xyz=0 -0.6 0 rpy=0 0 0
- joint scan_joint: origin xyz=0.0 0 1.2 rpy=0 0 0 -> xyz=0.0 0 0.6 rpy=0 0 0

Commit message: fixed a small error in scaling

File: src/bme_gazebo_sensors/urdf/mogi_bot.urdf (robot description, URDF)
Before this commit: robot mogi_bot, 8 links, 7 joints
Joints:
- joint camera_optical_joint: origin xyz=0 0 0 rpy=-0.78535 0 -0.78535 -> xyz=0 0 0 rpy=-1.5707 0 -1.5707

Commit message: new node for lane detection only . following yet to be done

File: src/bme_gazebo_sensors/urdf/mogi_bot.urdf (robot description, URDF)
Before this commit: robot mogi_bot, 8 links, 7 joints
Joints:
- joint camera_joint: origin xyz=0.9 0 0.3 rpy=0 0 0 -> xyz=0.9 0 1 rpy=0 0.2793 0

Commit message: inreased image resolution

File: src/bme_gazebo_sensors/urdf/mogi_bot.urdf (robot description, URDF)
Before this commit: robot mogi_bot, 8 links, 7 joints
Joints:
- joint camera_joint: origin xyz=0.9 0 0.3 rpy=0 0 0 -> xyz=0.9 0 1 rpy=0 0 0

Commit message: corrected point cloud orientation

File: src/bme_gazebo_sensors/urdf/mogi_bot.urdf (robot description, URDF)
Before this commit: robot mogi_bot, 8 links, 7 joints
Joints:
- joint camera_joint: origin xyz=0.9 0 1 rpy=0 0.2793 0 -> xyz=0.9 0 0.3 rpy=0 0.2793 0

Commit message: wide angle camera

File: src/bme_gazebo_sensors/urdf/mogi_bot.urdf (robot description, URDF)
Before this commit: robot mogi_bot, 8 links, 7 joints
Joints:
- joint camera_joint: origin xyz=0.9 0 0.3 rpy=0 0.2793 0 -> xyz=0.5 0 1.4 rpy=0 0 0

Commit message: lane following node implemented

File: src/bme_gazebo_sensors/urdf/mogi_bot.urdf (robot description, URDF)
Before this commit: robot mogi_bot, 8 links, 7 joints
Joints:
- joint camera_joint: origin xyz=0.9 0 0.3 rpy=0 0.2793 0 -> xyz=0.9 0 1 rpy=0 0.2793 0

Commit message: changed urdf

File: src/bme_gazebo_sensors/urdf/mogi_bot.urdf (robot description, URDF)
Before this commit: robot mogi_bot, 8 links, 7 joints
Links:
- removed link camera_link_optical
- removed link imu_link
- removed link left_wheel
- removed link right_wheel
- added link b_link, mass .1; collision cylinder length=.045 radius=.02; visual cylinder length=.045 radius=.02
- added link castor_back, mass 5.0; collision cylinder length=.03 radius=.06; visual cylinder length=.03 radius=.06
- added link castor_front, mass 5.0; collision cylinder length=.03 radius=.06; visual cylinder length=.03 radius=.06
- added link f_link, mass .1; collision cylinder length=.045 radius=.02; visual cylinder length=.045 radius=.02
- added link stick, mass 1.0; collision box size=.0625 .0625 .9; visual box size=.0625 .0625 .9
- added link wheel_left, mass 5.0; collision cylinder length=.1 radius=.1875; visual cylinder length=.1 radius=.1875
- added link wheel_right, mass 5.0; collision cylinder length=.1 radius=.1875; visual cylinder length=.1 radius=.1875
- link base_link: mass 30.0 -> 15.0; geometry collision box size=1.375 1 .35; visual box size=1.375 1 .35
- link camera_link: mass 0.1 -> 1.0; geometry collision box size=.075 .25 .075; visual box size=.075 .25 .075
- link scan_link: mass 1e-5 -> 1.0; geometry collision box size=.125 .125 .05; visual box size=.125 .125 .05
Joints:
- removed joint camera_joint
- removed joint camera_optical_joint
- removed joint imu_joint
- removed joint scan_joint
- added joint back_castor: type continuous, parent base_link, child castor_back, origin xyz=-.65 0 -.2775 rpy=0 0 0, axis 0 0 1, limit effort=100 velocity=10
- added joint camera: type fixed, parent stick, child camera_link, origin xyz=0 0 .45 rpy=0 0 0
- added joint front_castor: type continuous, parent base_link, child castor_front, origin xyz=.65 0 -.2775 rpy=0 0 0, axis 0 0 1, limit effort=100 velocity=10
- added joint lidar: type fixed, parent base_link, child scan_link, origin xyz=.59375 0 .3 rpy=0 0 0
- added joint linkb: type fixed, parent base_link, child b_link, origin xyz=-.65 0 -.19625 rpy=0 0 0
- added joint linkf: type fixed, parent base_link, child f_link, origin xyz=.65 0 -.19625 rpy=0 0 0
- added joint sensor_mount: type fixed, parent base_link, child stick, origin xyz=.4 0 .6 rpy=0 0 0
- joint base_footprint_joint: origin xyz=0 0 0 rpy=0 0 0 -> xyz=0 0 0.235 rpy=0 0 0
- joint left_wheel_joint: child left_wheel -> wheel_left; limit effort=100 velocity=80 -> effort=100 velocity=10; origin xyz=0 0.6 0 rpy=0 0 0 -> xyz=0 .55 -.15 rpy=0 0 0
- joint right_wheel_joint: child right_wheel -> wheel_right; origin xyz=0 -0.6 0 rpy=0 0 0 -> xyz=0 -.55 -.15 rpy=0 0 0

Commit message: fixed links for castor wheels and base_footprint

File: src/bme_gazebo_sensors/urdf/mogi_bot.urdf (robot description, URDF)
Before this commit: robot mogi_bot, 11 links, 10 joints
Links:
- link b_link: geometry collision cylinder length=.09 radius=.02; visual cylinder length=.09 radius=.02
- link f_link: geometry collision cylinder length=.09 radius=.02; visual cylinder length=.09 radius=.02
Joints:
- joint back_castor: origin xyz=-.65 0 -.2775 rpy=0 0 0 -> xyz=0 0 -.0825 rpy=0 0 0; parent base_link -> b_link
- joint base_footprint_joint: origin xyz=0 0 0.235 rpy=0 0 0 -> xyz=0 0 .375 rpy=0 0 0
- joint front_castor: origin xyz=.65 0 -.2775 rpy=0 0 0 -> xyz=0 0 -.0825 rpy=0 0 0; parent base_link -> f_link
- joint left_wheel_joint: origin xyz=0 .55 -.15 rpy=0 0 0 -> xyz=0 .55 -0.1875 rpy=0 0 0
- joint linkb: origin xyz=-.65 0 -.19625 rpy=0 0 0 -> xyz=-.65 0 -.2 rpy=0 0 0
- joint linkf: origin xyz=.65 0 -.19625 rpy=0 0 0 -> xyz=.65 0 -.2 rpy=0 0 0
- joint right_wheel_joint: origin xyz=0 -.55 -.15 rpy=0 0 0 -> xyz=0 -.55 -0.1875 rpy=0 0 0

Commit message: l

File: src/bme_gazebo_sensors/urdf/mogi_bot.urdf (robot description, URDF)
Before this commit: robot mogi_bot, 11 links, 10 joints
Links:
- removed link stick
Joints:
- removed joint sensor_mount
- joint back_castor: parent base_link -> b_link
- joint camera: parent stick -> base_link
- joint front_castor: parent base_link -> f_link

Commit message: blahblahblah

File: src/bme_gazebo_sensors/urdf/mogi_bot.urdf (robot description, URDF)
Before this commit: robot mogi_bot, 11 links, 10 joints
Links:
- link b_link: geometry collision cylinder length=.15 radius=.02; visual cylinder length=.15 radius=.02
- link f_link: geometry collision cylinder length=.15 radius=.02; visual cylinder length=.15 radius=.02
Joints:
- joint back_castor: origin xyz=-.65 0 -.2775 rpy=0 0 0 -> xyz=0 0 -.115 rpy=0 0 0; parent base_link -> b_link
- joint base_footprint_joint: origin xyz=0 0 0.235 rpy=0 0 0 -> xyz=0 0 .375 rpy=0 0 0
- joint front_castor: origin xyz=.65 0 -.2775 rpy=0 0 0 -> xyz=0 0 -.115 rpy=0 0 0; parent base_link -> f_link
- joint left_wheel_joint: origin xyz=0 .55 -.15 rpy=0 0 0 -> xyz=0 .55 -0.1875 rpy=0 0 0
- joint linkb: origin xyz=-.65 0 -.19625 rpy=0 0 0 -> xyz=-.65 0 -.2 rpy=0 0 0
- joint linkf: origin xyz=.65 0 -.19625 rpy=0 0 0 -> xyz=.65 0 -.2 rpy=0 0 0
- joint right_wheel_joint: origin xyz=0 -.55 -.15 rpy=0 0 0 -> xyz=0 -.55 -0.1875 rpy=0 0 0

Commit message: Idk

File: src/bme_gazebo_sensors/urdf/mogi_bot.urdf (robot description, URDF)
Before this commit: robot mogi_bot, 12 links, 11 joints
Links:
- added link bcamera_link, mass 1.0; collision box size=.075 .25 .075; visual box size=.075 .25 .075
Joints:
- added joint bcamera: type fixed, parent stick, child bcamera_link, origin xyz=-0.75 0 0.45 rpy=0 0 3.1416

Commit message: proper yellow lane centre detection

File: src/bme_gazebo_sensors/urdf/mogi_bot.urdf (robot description, URDF)
Before this commit: robot mogi_bot, 11 links, 10 joints
Links:
- added link bcamera_link, mass 1.0; collision box size=.075 .25 .075; visual box size=.075 .25 .075
- added link navsat_link
Joints:
- added joint bcamera: type fixed, parent stick, child bcamera_link, origin xyz=-0.75 0 0.45 rpy=0 0 3.1416
- added joint navsat_joint: type fixed, parent base_link, child navsat_link, origin xyz=0 0 0 rpy=0 0 0

Commit message: added gpu based dbscan

File: src/bme_gazebo_sensors/urdf/mogi_bot.urdf (robot description, URDF)
Before this commit: robot mogi_bot, 10 links, 9 joints
Links:
- added link stick, mass 1.0; collision box size=.0625 .0625 .9; visual box size=.0625 .0625 .9
Joints:
- added joint sensor_mount: type fixed, parent base_link, child stick, origin xyz=.4 0 .6 rpy=0 0 0
- joint camera: parent base_link -> stick
