Commit message: finished controller

File: src/igvc/urdf/mogi_bot.urdf (robot description, URDF)
Before this commit: robot mogi_bot, 13 links, 12 joints
Links:
- added link imu_link, mass 0.001
Joints:
- added joint camera_to_imu: type fixed, parent camera_link, child imu_link, origin xyz=0 0 0 rpy=0 0 0

Commit message: added lidar

File: src/igvc/urdf/mogi_bot.urdf (robot description, URDF)
Before this commit: robot mogi_bot, 14 links, 13 joints
Links:
- link scan_link: mass 1.0 -> 1e-5; geometry collision box size=.1 .1 .1; visual mesh filename=package://igvc/meshes/lidar.dae
Joints:
- removed joint lidar
- added joint scan_joint: type fixed, parent base_link, child scan_link, origin xyz=0.0 0 0.15 rpy=0 0 0, axis 0 1 0

Commit message: please work

File: src/igvc/urdf/mogi_bot.urdf (robot description, URDF)
Before this commit: robot mogi_bot, 14 links, 13 joints
Links:
- added link stereo_left_camera_link, mass 1.0; collision box size=.075 .25 .075; visual box size=.075 .25 .075
- added link stereo_right_camera_link, mass 1.0; collision box size=.075 .25 .075; visual box size=.075 .25 .075
Joints:
- added joint stereo_left_camera_joint: type fixed, parent stick, child stereo_left_camera_link, origin xyz=0.0 0.05 0.45 rpy=0 0 0
- added joint stereo_right_camera_joint: type fixed, parent stick, child stereo_right_camera_link, origin xyz=0.0 -0.05 0.45 rpy=0 0 0

Commit message: Revert "Merge branch 'main' of github.com:Team-Abhiyaan/igvc-sim"
This reverts commit 2c1e4a0fa3a5f2c3007579703cbf74485daa7c2e, reversing
changes made to e3311d865a611ab7647bb87e4ab4b9f17eda2908.

File: src/igvc/urdf/mogi_bot.urdf (robot description, URDF)
Before this commit: robot mogi_bot, 16 links, 15 joints
Links:
- link scan_link: mass 1e-5 -> 1.0; geometry collision box size=.125 .125 .05; visual box size=.125 .125 .05
Joints:
- removed joint scan_joint
- added joint lidar: type fixed, parent base_link, child scan_link, origin xyz=.59375 0 .3 rpy=0 0 0

Commit message: fixed world, added new ground plane for autonav

File: src/igvc/urdf/mogi_bot.urdf (robot description, URDF)
Before this commit: robot mogi_bot, 16 links, 15 joints
Links:
- removed link stereo_left_camera_link
- removed link stereo_right_camera_link
Joints:
- removed joint stereo_left_camera_joint
- removed joint stereo_right_camera_joint

Commit message: Added pitch wooo

File: src/igvc/urdf/mogi_bot.urdf (robot description, URDF)
Before this commit: robot mogi_bot, 14 links, 13 joints
Links:
- link stick: geometry collision box size=.0325 .0325 .8; visual box size=.0325 .0325 .8
Joints:
- joint camera: origin xyz=0 0 .45 rpy=0 0 0 -> xyz=0 0 .45 rpy=0 .38 0
